File: SenseEHajo.kicad_sch (KiCad schematic)
At the start: 103 parts, among them IC1 AP3012, IC2 MCP3221, IC3 74LVC1G125, IC4 K814P, IC5 74LVC1G125, IC6 74LVC1G125, IC7 74LVC1G10, J1 Conn_01x02_Male, J2 REED, J3 RTC ( DS3231)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

Commit message: Fix Display BTP senese for press
Parts:
- removed R36: 10k, Resistor_SMD:R_0805_2012Metric_Pad1.20x1.40mm_HandSolder, symbol Device:R_Small
- removed R37: 1k, Resistor_SMD:R_0805_2012Metric_Pad1.20x1.40mm_HandSolder, symbol Device:R_Small
- removed U5: MCP6001-OT, Package_TO_SOT_SMD:SOT-23-5, symbol Amplifier_Operational:MCP6001-OT
- added F1: 0.5A / 230VAC, Capacitor_THT:C_Rect_L7.0mm_W4.5mm_P5.00mm, symbol Device:Fuse
- added IC8: INA350ABS, Package_TO_SOT_SMD:SOT-23-8_Handsoldering, symbol TI:INA350ABS
- added IO15, IO19, IO2, IO21, IO32, IO33, IO34, IO35, S_VN1, S_VP1: IO32, TestPoint:TestPoint_Pad_D2.0mm, symbol Connector:TestPoint
- added RV1: Varistor 10D561, Varistor:RV_Disc_D9mm_W5.2mm_P5mm, symbol Device:Varistor
- added TP3: I2C_DISP_SDA_3V3, TestPoint:TestPoint_Pad_D2.0mm, symbol Connector:TestPoint
- added TP4: I2C_DISP_SCL_3V3, TestPoint:TestPoint_Pad_D2.0mm, symbol Connector:TestPoint
- added TP5: 3V3, TestPoint:TestPoint_Pad_D2.0mm, symbol Connector:TestPoint
- added TP6: 5V, TestPoint:TestPoint_Pad_D2.0mm, symbol Connector:TestPoint
- added TP7: MAINS Halvewaves, TestPoint:TestPoint_Pad_D2.0mm, symbol Connector:TestPoint
- added TP8: 12V, TestPoint:TestPoint_Pad_D2.0mm, symbol Connector:TestPoint
Connections:
- net +12V: now also TP8.1
- net +3V3: now also TP5.1
- net +5V: now also IC8.7 (V+), IC8.8 (SHDN), TP6.1
- net GND: now also IC8.1 (GS), IC8.4 (V-), IC8.5 (REF)
- net I2C_DSP_SCL: now also TP4.1
- net I2C_DSP_SDA: now also TP3.1
- net L_230V: now also F1.1; no longer PS1.1 (AC/L)
- net MAINS_HALVEWAVES: now also TP7.1
- net N_230V: now also RV1.1
- net SCL_DSP: now also IC8.2 (IN-)
- net at U1.23 (IO15): now also IO15.1
- net at U1.24 (IO2): now also IO2.1
- net at U1.31 (IO19): now also IO19.1
- net at U1.33 (IO21): now also IO21.1
- net at U1.4 (SENSOR_VP): now also S_VP1.1
- net at U1.5 (SENSOR_VN): now also S_VN1.1
- net at U1.6 (IO34): now also IO34.1
- net at U1.7 (IO35): now also IO35.1
- net at U1.8 (IO32): now also IO32.1
- net at U1.9 (IO33): now also IO33.1
- net at IC6.2 (A): now also IC8.6 (OUT)
- net at IC5.4 (Y), R29.2: now also IC8.3 (IN+)
- new net: F1.2, PS1.1 (AC/L), RV1.2
Other:
- note added: "Add common mode choke here ~10uH + 100nF Cap"
- note added: "For I2C Transfer we have > 10k input impedance This means we will get with 100R Shunt ~0.5mA current This results in 0,05V drop and with the INA350 we get ~0,5V Vout. The 74LVC1G125 needs 0.8V to detect a logic high"
- note added: "INA350 is a instrumentational amp with G=10 With ~0.22V we will get 2,2V output"
- note added: "use isolated supply"
- note removed: "Add fuse here later"
- note removed: "ISOLATED supply can be replaced with OFFLINE AC/DC converter"
- note removed: "If BL0937 powermeter shall be used als use non isolated supply"
- note removed: "OPV output is R2/R1+1 = 10k/1k+1=11 With ~0.22V we will get 2,42V output"
- note removed: "PCB may float on mains"
- moved on the sheet: C11, C27, C9, IC4, J7, J8, PS1, R29, R5, R6, R7, U6
